Commit message: Fix iiwa 14 dimensions

File: kuka_lbr_iiwa_support/urdf/lbr_iiwa14_r820_macro.xacro (robot description, xacro)
@@ -131,5 +131,5 @@
       <parent link="${prefix}base_link"/>
       <child link="${prefix}link_1"/>
-      <origin rpy="-0.0 0.0 0.0" xyz="0.0 0.0 0.1375"/>
+      <origin rpy="-0.0 0.0 0.0" xyz="0.0 0.0 0.1395"/>
       <axis xyz="0.0 0.0 1.0"/>
       <limit effort="0" lower="${radians(-170)}" upper="${radians(170)}" velocity="${radians(85)}"/>
@@ -145,5 +145,5 @@
       <parent link="${prefix}link_2"/>
       <child link="${prefix}link_3"/>
-      <origin rpy="-0.0 0.0 0.0" xyz="0.0 0.0 0.1845"/>
+      <origin rpy="-0.0 0.0 0.0" xyz="0.0 0.0 0.1865"/>
       <axis xyz="0.0 0.0 1.0"/>
       <limit effort="0" lower="${radians(-170)}" upper="${radians(170)}" velocity="${radians(100)}"/>

Commit message: Actually fix the dimensions

File: kuka_lbr_iiwa_support/urdf/lbr_iiwa14_r820_macro.xacro (robot description, xacro)
@@ -131,5 +131,5 @@
       <parent link="${prefix}base_link"/>
       <child link="${prefix}link_1"/>
-      <origin rpy="-0.0 0.0 0.0" xyz="0.0 0.0 0.1395"/>
+      <origin rpy="-0.0 0.0 0.0" xyz="0.0 0.0 0.1575"/>
       <axis xyz="0.0 0.0 1.0"/>
       <limit effort="0" lower="${radians(-170)}" upper="${radians(170)}" velocity="${radians(85)}"/>
@@ -145,5 +145,5 @@
       <parent link="${prefix}link_2"/>
       <child link="${prefix}link_3"/>
-      <origin rpy="-0.0 0.0 0.0" xyz="0.0 0.0 0.1865"/>
+      <origin rpy="-0.0 0.0 0.0" xyz="0.0 0.0 0.2045"/>
       <axis xyz="0.0 0.0 1.0"/>
       <limit effort="0" lower="${radians(-170)}" upper="${radians(170)}" velocity="${radians(100)}"/>

Commit message: Now in technicolor

File: kuka_lbr_iiwa_support/urdf/lbr_iiwa14_r820_macro.xacro (robot description, xacro)
@@ -13,5 +13,5 @@
       <visual>
         <geometry>
-          <mesh filename="package://kuka_lbr_iiwa_support/meshes/lbr_iiwa14_r820/visual/base_link.stl"/>
+          <mesh filename="package://kuka_lbr_iiwa_support/meshes/lbr_iiwa14_r820/visual/base_link.dae"/>
         </geometry>
         <origin rpy="-0.0 0.0 0.0" xyz="0.0 0.0 0.0"/>
@@ -27,5 +27,5 @@
       <visual>
         <geometry>
-          <mesh filename="package://kuka_lbr_iiwa_support/meshes/lbr_iiwa14_r820/visual/link_1.stl"/>
+          <mesh filename="package://kuka_lbr_iiwa_support/meshes/lbr_iiwa14_r820/visual/link_1.dae"/>
         </geometry>
         <origin rpy="-0.0 0.0 0.0" xyz="0.0 0.0 0.0"/>
@@ -41,5 +41,5 @@
       <visual>
         <geometry>
-          <mesh filename="package://kuka_lbr_iiwa_support/meshes/lbr_iiwa14_r820/visual/link_2.stl"/>
+          <mesh filename="package://kuka_lbr_iiwa_support/meshes/lbr_iiwa14_r820/visual/link_2.dae"/>
         </geometry>
         <origin rpy="-0.0 0.0 0.0" xyz="0.0 0.0 0.0"/>
@@ -55,5 +55,5 @@
       <visual>
         <geometry>
-          <mesh filename="package://kuka_lbr_iiwa_support/meshes/lbr_iiwa14_r820/visual/link_3.stl"/>
+          <mesh filename="package://kuka_lbr_iiwa_support/meshes/lbr_iiwa14_r820/visual/link_3.dae"/>
         </geometry>
         <origin rpy="-0.0 0.0 0.0" xyz="0.0 0.0 0.0"/>
@@ -69,5 +69,5 @@
       <visual>
         <geometry>
-          <mesh filename="package://kuka_lbr_iiwa_support/meshes/lbr_iiwa14_r820/visual/link_4.stl"/>
+          <mesh filename="package://kuka_lbr_iiwa_support/meshes/lbr_iiwa14_r820/visual/link_4.dae"/>
         </geometry>
         <origin rpy="-0.0 0.0 0.0" xyz="0.0 0.0 0.0"/>
@@ -83,5 +83,5 @@
       <visual>
         <geometry>
-          <mesh filename="package://kuka_lbr_iiwa_support/meshes/lbr_iiwa14_r820/visual/link_5.stl"/>
+          <mesh filename="package://kuka_lbr_iiwa_support/meshes/lbr_iiwa14_r820/visual/link_5.dae"/>
         </geometry>
         <origin rpy="-0.0 0.0 0.0" xyz="0.0 0.0 0.0"/>
@@ -97,5 +97,5 @@
       <visual>
         <geometry>
-          <mesh filename="package://kuka_lbr_iiwa_support/meshes/lbr_iiwa14_r820/visual/link_6.stl"/>
+          <mesh filename="package://kuka_lbr_iiwa_support/meshes/lbr_iiwa14_r820/visual/link_6.dae"/>
         </geometry>
         <origin rpy="-0.0 0.0 0.0" xyz="0.0 0.0 0.0"/>
@@ -111,5 +111,5 @@
       <visual>
         <geometry>
-          <mesh filename="package://kuka_lbr_iiwa_support/meshes/lbr_iiwa14_r820/visual/link_7.stl"/>
+          <mesh filename="package://kuka_lbr_iiwa_support/meshes/lbr_iiwa14_r820/visual/link_7.dae"/>
         </geometry>
         <origin rpy="-0.0 0.0 0.0" xyz="0.0 0.0 0.0"/>
